Commit message: Moving to v4

File: arm2d2_v2_description/urdf/arm2d2.urdf (robot description, URDF)
Before this commit: robot arm2d2, 11 links, 10 joints
Links:
- link actuator_1: geometry collision mesh filename=package://arm2d2_v2_description/meshes/actuator_1_2.stl scale=0.001 0.001 0.001; visual mesh filename=package://arm2d2_v2_description/meshes/actuator_1_2.stl scale=0.001 0.001 0.001
- link actuator_2: geometry collision mesh filename=package://arm2d2_v2_description/meshes/actuator_2_1.stl scale=0.001 0.001 0.001; visual mesh filename=package://arm2d2_v2_description/meshes/actuator_2_1.stl scale=0.001 0.001 0.001
- link actuator_3: geometry collision mesh filename=package://arm2d2_v2_description/meshes/actuator_3_1.stl scale=0.001 0.001 0.001; visual mesh filename=package://arm2d2_v2_description/meshes/actuator_3_1.stl scale=0.001 0.001 0.001

File: arm2d2_v2_description/urdf/arm2d2.urdf.xacro (robot description, xacro)
@@ -20,5 +20,5 @@
         <origin xyz="0 0 0.0025" rpy="0 0 0"/>
         <geometry>
-        <mesh filename="package://arm2d2_description/meshes/base_plate.stl" scale="0.001 0.001 0.001"/>
+        <mesh filename="package://arm2d2_v2_description/meshes/base_plate.stl" scale="0.001 0.001 0.001"/>
         </geometry>
         <material name="silver"/>
@@ -27,5 +27,5 @@
         <origin xyz="0 0 0.0025" rpy="0 0 0"/>
         <geometry>
-        <mesh filename="package://arm2d2_description/meshes/base_plate.stl" scale="0.001 0.001 0.001"/>
+        <mesh filename="package://arm2d2_v2_description/meshes/base_plate.stl" scale="0.001 0.001 0.001"/>
         </geometry>
     </collision>
@@ -70,5 +70,5 @@
       <origin xyz="-0.0851 -0.006604 0.0851" rpy="0 0 0"/>
       <geometry>
-        <mesh filename="package://arm2d2_description/meshes/link_1_1.stl" scale="0.001 0.001 0.001"/>
+        <mesh filename="package://arm2d2_v2_description/meshes/link_1_1.stl" scale="0.001 0.001 0.001"/>
       </geometry>
       <material name="silver"/>
@@ -77,5 +77,5 @@
       <origin xyz="-0.0851 -0.006604 0.0851" rpy="0 0 0"/>
       <geometry>
-        <mesh filename="package://arm2d2_description/meshes/link_1_1.stl" scale="0.001 0.001 0.001"/>
+        <mesh filename="package://arm2d2_v2_description/meshes/link_1_1.stl" scale="0.001 0.001 0.001"/>
       </geometry>
     </collision>
@@ -97,5 +97,5 @@
       <origin xyz="-0.090305 -0.046604 0.085785" rpy="0 0 0"/>
       <geometry>
-        <mesh filename="package://arm2d2_description/meshes/link_2_1.stl" scale="0.001 0.001 0.001"/>
+        <mesh filename="package://arm2d2_v2_description/meshes/link_2_1.stl" scale="0.001 0.001 0.001"/>
       </geometry>
       <material name="silver"/>
@@ -104,5 +104,5 @@
       <origin xyz="-0.090305 -0.046604 0.085785" rpy="0 0 0"/>
       <geometry>
-        <mesh filename="package://arm2d2_description/meshes/link_2_1.stl" scale="0.001 0.001 0.001"/>
+        <mesh filename="package://arm2d2_v2_description/meshes/link_2_1.stl" scale="0.001 0.001 0.001"/>
       </geometry>
     </collision>
@@ -124,5 +124,5 @@
       <origin xyz="-0.084346 -0.183285 0.054438" rpy="0 0 0"/>
       <geometry>
-        <mesh filename="package://arm2d2_description/meshes/link_3_1.stl" scale="0.001 0.001 0.001"/>
+        <mesh filename="package://arm2d2_v2_description/meshes/link_3_1.stl" scale="0.001 0.001 0.001"/>
       </geometry>
       <material name="silver"/>
@@ -131,5 +131,5 @@
       <origin xyz="-0.084346 -0.183285 0.054438" rpy="0 0 0"/>
       <geometry>
-        <mesh filename="package://arm2d2_description/meshes/link_3_1.stl" scale="0.001 0.001 0.001"/>
+        <mesh filename="package://arm2d2_v2_description/meshes/link_3_1.stl" scale="0.001 0.001 0.001"/>
       </geometry>
     </collision>
@@ -151,5 +151,5 @@
       <origin xyz="-0.059366 -0.168718 0.013574" rpy="0 0 0"/>
       <geometry>
-        <mesh filename="package://arm2d2_description/meshes/link_4_1.stl" scale="0.001 0.001 0.001"/>
+        <mesh filename="package://arm2d2_v2_description/meshes/link_4_1.stl" scale="0.001 0.001 0.001"/>
       </geometry>
       <material name="silver"/>
@@ -158,5 +158,5 @@
       <origin xyz="-0.059366 -0.168718 0.013574" rpy="0 0 0"/>
       <geometry>
-        <mesh filename="package://arm2d2_description/meshes/link_4_1.stl" scale="0.001 0.001 0.001"/>
+        <mesh filename="package://arm2d2_v2_description/meshes/link_4_1.stl" scale="0.001 0.001 0.001"/>
       </geometry>
     </collision>
@@ -178,5 +178,5 @@
       <origin xyz="-0.091433 -0.131975 -0.076012" rpy="0 0 0"/>
       <geometry>
-        <mesh filename="package://arm2d2_description/meshes/link_5_1.stl" scale="0.001 0.001 0.001"/>
+        <mesh filename="package://arm2d2_v2_description/meshes/link_5_1.stl" scale="0.001 0.001 0.001"/>
       </geometry>
       <material name="silver"/>
@@ -185,5 +185,5 @@
       <origin xyz="-0.091433 -0.131975 -0.076012" rpy="0 0 0"/>
       <geometry>
-        <mesh filename="package://arm2d2_description/meshes/link_5_1.stl" scale="0.001 0.001 0.001"/>
+        <mesh filename="package://arm2d2_v2_description/meshes/link_5_1.stl" scale="0.001 0.001 0.001"/>
       </geometry>
     </collision>
@@ -205,5 +205,5 @@
     <origin xyz="0 0 0" rpy="0 0 0"/>
     <geometry>
-      <mesh filename="package://arm2d2_description/meshes/palm.stl" scale="0.001 0.001 0.001"/>
+      <mesh filename="package://arm2d2_v2_description/meshes/palm.stl" scale="0.001 0.001 0.001"/>
     </geometry>
     <material name="silver"/>
@@ -212,5 +212,5 @@
     <origin xyz="0 0 0" rpy="0 0 0"/>
     <geometry>
-      <mesh filename="package://arm2d2_description/meshes/palm.stl" scale="0.001 0.001 0.001"/>
+      <mesh filename="package://arm2d2_v2_description/meshes/palm.stl" scale="0.001 0.001 0.001"/>
     </geometry>
   </collision>
@@ -244,5 +244,5 @@
       <origin xyz="-0.008797 0.014908 -0.021091" rpy="0 0 0"/>
       <geometry>
-        <mesh filename="package://arm2d2_description/meshes/actuator_1_2.stl" scale="0.001 0.001 0.001"/>
+        <mesh filename="package://arm2d2_v2_description/meshes/actuator_1_2.stl" scale="0.001 0.001 0.001"/>
       </geometry>
       <material name="silver"/>
@@ -251,5 +251,5 @@
       <origin xyz="-0.008797 0.014908 -0.021091" rpy="0 0 0"/>
       <geometry>
-        <mesh filename="package://arm2d2_description/meshes/actuator_1_2.stl" scale="0.001 0.001 0.001"/>
+        <mesh filename="package://arm2d2_v2_description/meshes/actuator_1_2.stl" scale="0.001 0.001 0.001"/>
       </geometry>
     </collision>
@@ -271,5 +271,5 @@
         <origin xyz="-0.013822 0.015067 0.017999" rpy="0 0 0"/>
         <geometry>
-          <mesh filename="package://arm2d2_description/meshes/actuator_2_1.stl" scale="0.001 0.001 0.001"/>
+          <mesh filename="package://arm2d2_v2_description/meshes/actuator_2_1.stl" scale="0.001 0.001 0.001"/>
         </geometry>
         <material name="silver"/>
@@ -278,5 +278,5 @@
         <origin xyz="-0.013822 0.015067 0.017999" rpy="0 0 0"/>
         <geometry>
-          <mesh filename="package://arm2d2_description/meshes/actuator_2_1.stl" scale="0.001 0.001 0.001"/>
+          <mesh filename="package://arm2d2_v2_description/meshes/actuator_2_1.stl" scale="0.001 0.001 0.001"/>
         </geometry>
       </collision>
@@ -298,5 +298,5 @@
         <origin xyz="0.022563 0.015024 0.00279" rpy="0 0 0"/>
         <geometry>
-          <mesh filename="package://arm2d2_description/meshes/actuator_3_1.stl" scale="0.001 0.001 0.001"/>
+          <mesh filename="package://arm2d2_v2_description/meshes/actuator_3_1.stl" scale="0.001 0.001 0.001"/>
         </geometry>
         <material name="silver"/>
@@ -305,5 +305,5 @@
         <origin xyz="0.022563 0.015024 0.00279" rpy="0 0 0"/>
         <geometry>
-          <mesh filename="package://arm2d2_description/meshes/actuator_3_1.stl" scale="0.001 0.001 0.001"/>
+          <mesh filename="package://arm2d2_v2_description/meshes/actuator_3_1.stl" scale="0.001 0.001 0.001"/>
         </geometry>
       </collision>

File: arm2d2_v3_description/urdf/arm2d2.urdf.xacro (robot description, xacro)
@@ -130,5 +130,5 @@
   </collision>
 </link>
-<link name="gripper_1">
+<link name="gripper">
   <inertial>
     <origin xyz="0.0005651763785821801 0.06065258242303184 0.01133988363017737" rpy="0 0 0"/>
@@ -139,5 +139,5 @@
     <origin xyz="0.110082 -0.292458 0.066268" rpy="0 0 0"/>
     <geometry>
-      <mesh filename="package://arm2d2_v3_description/meshes/gripper_1.stl" scale="0.01 0.01 0.01"/>
+      <mesh filename="package://arm2d2_v3_description/meshes/gripper.stl" scale="0.01 0.01 0.01"/>
     </geometry>
     <material name="silver"/>
@@ -146,5 +146,5 @@
     <origin xyz="0.110082 -0.292458 0.066268" rpy="0 0 0"/>
     <geometry>
-      <mesh filename="package://arm2d2_v3_description/meshes/gripper_1.stl" scale="0.01 0.01 0.01"/>
+      <mesh filename="package://arm2d2_v3_description/meshes/gripper.stl" scale="0.01 0.01 0.01"/>
     </geometry>
   </collision>
@@ -185,5 +185,5 @@
   <origin xyz="0.0 0.035617 -0.01" rpy="0 0 0"/>
   <parent link="link_5"/>
-  <child link="gripper_1"/>
+  <child link="gripper"/>
   <axis xyz="0.0 -0.0 -1.0"/>
   <limit upper="1.919862" lower="-1.919862" effort="100" velocity="100"/>
