Commit message: 7DOF mostly works

File: arm2v4_description/urdf/arm2v4.urdf.xacro (robot description, xacro)
@@ -1,7 +1,8 @@
 <?xml version="1.0" ?>
-<robot name="arm2_v4" xmlns:xacro="http://www.ros.org/wiki/xacro">
-<xacro:include filename="$(find arm2_v4_description)/urdf/materials.xacro" />
-<xacro:include filename="$(find arm2_v4_description)/urdf/arm2_v4.trans" />
-<xacro:include filename="$(find arm2_v4_description)/urdf/arm2_v4.gazebo" />
+<robot name="arm2v4" xmlns:xacro="http://www.ros.org/wiki/xacro">
+<material name="silver">
+  <color rgba="0.700 0.700 0.700 1.000" />
+</material>
+<link name="world"/>
 <link name="base_link">
   <inertial>
@@ -13,5 +14,5 @@
     <origin xyz="0 0 0" rpy="0 0 0"/>
     <geometry>
-      <mesh filename="package://arm2_v4_description/meshes/base_link.stl" scale="0.001 0.001 0.001"/>
+      <mesh filename="package://arm2v4_description/meshes/base_link.stl" scale="0.01 0.01 0.01"/>
     </geometry>
     <material name="silver"/>
@@ -20,8 +21,38 @@
     <origin xyz="0 0 0" rpy="0 0 0"/>
     <geometry>
-      <mesh filename="package://arm2_v4_description/meshes/base_link.stl" scale="0.001 0.001 0.001"/>
-    </geometry>
-  </collision>
-</link>
+      <mesh filename="package://arm2v4_description/meshes/base_link.stl" scale="0.01 0.01 0.01"/>
+    </geometry>
+  </collision>
+</link>
+<joint name="world_joint" type="fixed">
+  <parent link="world"/>
+  <child link="base_link"/>
+  <origin xyz="0 0 0" rpy="1.57 0 0"/>
+</joint>
+  <link name="top_plate">
+    <inertial>
+        <origin xyz="-2.154281413321998e-06 0.0035387814754625734 -0.0056639470834143136" rpy="0 0 0"/>
+        <mass value="1.5479093566761954"/>
+        <inertia ixx="0.010238" iyy="0.01139" izz="0.021617" ixy="-0.0" iyz="0.0" ixz="0.0"/>
+    </inertial>
+    <visual>
+        <origin xyz="0 0 0" rpy="0 0 0"/>
+        <geometry>
+        <mesh filename="package://arm2d2_v2_description/meshes/base_plate.stl" scale="0.001 0.001 0.001"/>
+        </geometry>
+        <material name="silver"/>
+    </visual>
+    <collision>
+        <origin xyz="0 0 0.279654" rpy="0 0 0"/>
+        <geometry>
+        <mesh filename="package://arm2d2_v2_description/meshes/base_plate.stl" scale="0.001 0.001 0.001"/>
+        </geometry>
+    </collision>
+  </link>
+  <joint name="top_connector" type="fixed">
+    <parent link="world"/>
+    <child link="top_plate"/>
+    <origin xyz="0 0 0.279654" rpy="0 0 0"/>
+  </joint>
 <link name="link_1">
   <inertial>
@@ -33,5 +64,5 @@
     <origin xyz="0.1101 -0.00635 0.0551" rpy="0 0 0"/>
     <geometry>
-      <mesh filename="package://arm2_v4_description/meshes/link_1.stl" scale="0.001 0.001 0.001"/>
+      <mesh filename="package://arm2v4_description/meshes/link_1.stl" scale="0.01 0.01 0.01"/>
     </geometry>
     <material name="silver"/>
@@ -40,5 +71,5 @@
     <origin xyz="0.1101 -0.00635 0.0551" rpy="0 0 0"/>
     <geometry>
-      <mesh filename="package://arm2_v4_description/meshes/link_1.stl" scale="0.001 0.001 0.001"/>
+      <mesh filename="package://arm2v4_description/meshes/link_1.stl" scale="0.01 0.01 0.01"/>
     </geometry>
   </collision>
@@ -53,5 +84,5 @@
     <origin xyz="0.1101 -0.041967 0.0581" rpy="0 0 0"/>
     <geometry>
-      <mesh filename="package://arm2_v4_description/meshes/link_2.stl" scale="0.001 0.001 0.001"/>
+      <mesh filename="package://arm2v4_description/meshes/link_2.stl" scale="0.01 0.01 0.01"/>
     </geometry>
     <material name="silver"/>
@@ -60,5 +91,5 @@
     <origin xyz="0.1101 -0.041967 0.0581" rpy="0 0 0"/>
     <geometry>
-      <mesh filename="package://arm2_v4_description/meshes/link_2.stl" scale="0.001 0.001 0.001"/>
+      <mesh filename="package://arm2v4_description/meshes/link_2.stl" scale="0.01 0.01 0.01"/>
     </geometry>
   </collision>
@@ -73,5 +104,5 @@
     <origin xyz="0.1101 -0.130967 0.0551" rpy="0 0 0"/>
     <geometry>
-      <mesh filename="package://arm2_v4_description/meshes/link_3.stl" scale="0.001 0.001 0.001"/>
+      <mesh filename="package://arm2v4_description/meshes/link_3.stl" scale="0.01 0.01 0.01"/>
     </geometry>
     <material name="silver"/>
@@ -80,5 +111,5 @@
     <origin xyz="0.1101 -0.130967 0.0551" rpy="0 0 0"/>
     <geometry>
-      <mesh filename="package://arm2_v4_description/meshes/link_3.stl" scale="0.001 0.001 0.001"/>
+      <mesh filename="package://arm2v4_description/meshes/link_3.stl" scale="0.01 0.01 0.01"/>
     </geometry>
   </collision>
@@ -93,5 +124,5 @@
     <origin xyz="0.1101 -0.166585 0.0581" rpy="0 0 0"/>
     <geometry>
-      <mesh filename="package://arm2_v4_description/meshes/link_4.stl" scale="0.001 0.001 0.001"/>
+      <mesh filename="package://arm2v4_description/meshes/link_4.stl" scale="0.01 0.01 0.01"/>
     </geometry>
     <material name="silver"/>
@@ -100,5 +131,5 @@
     <origin xyz="0.1101 -0.166585 0.0581" rpy="0 0 0"/>
     <geometry>
-      <mesh filename="package://arm2_v4_description/meshes/link_4.stl" scale="0.001 0.001 0.001"/>
+      <mesh filename="package://arm2v4_description/meshes/link_4.stl" scale="0.01 0.01 0.01"/>
     </geometry>
   </collision>
@@ -113,5 +144,5 @@
     <origin xyz="0.1101 -0.255585 0.0551" rpy="0 0 0"/>
     <geometry>
-      <mesh filename="package://arm2_v4_description/meshes/link_5.stl" scale="0.001 0.001 0.001"/>
+      <mesh filename="package://arm2v4_description/meshes/link_5.stl" scale="0.01 0.01 0.01"/>
     </geometry>
     <material name="silver"/>
@@ -120,5 +151,5 @@
     <origin xyz="0.1101 -0.255585 0.0551" rpy="0 0 0"/>
     <geometry>
-      <mesh filename="package://arm2_v4_description/meshes/link_5.stl" scale="0.001 0.001 0.001"/>
+      <mesh filename="package://arm2v4_description/meshes/link_5.stl" scale="0.01 0.01 0.01"/>
     </geometry>
   </collision>
@@ -133,5 +164,5 @@
     <origin xyz="0.1101 -0.291202 0.0581" rpy="0 0 0"/>
     <geometry>
-      <mesh filename="package://arm2_v4_description/meshes/link_6.stl" scale="0.001 0.001 0.001"/>
+      <mesh filename="package://arm2v4_description/meshes/link_6.stl" scale="0.01 0.01 0.01"/>
     </geometry>
     <material name="silver"/>
@@ -140,5 +171,5 @@
     <origin xyz="0.1101 -0.291202 0.0581" rpy="0 0 0"/>
     <geometry>
-      <mesh filename="package://arm2_v4_description/meshes/link_6.stl" scale="0.001 0.001 0.001"/>
+      <mesh filename="package://arm2v4_description/meshes/link_6.stl" scale="0.01 0.01 0.01"/>
     </geometry>
   </collision>
@@ -153,5 +184,5 @@
     <origin xyz="0.1101 -0.380202 0.0551" rpy="0 0 0"/>
     <geometry>
-      <mesh filename="package://arm2_v4_description/meshes/gripper.stl" scale="0.001 0.001 0.001"/>
+      <mesh filename="package://arm2v4_description/meshes/gripper.stl" scale="0.01 0.01 0.01"/>
     </geometry>
     <material name="silver"/>
@@ -160,9 +191,9 @@
     <origin xyz="0.1101 -0.380202 0.0551" rpy="0 0 0"/>
     <geometry>
-      <mesh filename="package://arm2_v4_description/meshes/gripper.stl" scale="0.001 0.001 0.001"/>
-    </geometry>
-  </collision>
-</link>
-<joint name="joint" type="revolute">
+      <mesh filename="package://arm2v4_description/meshes/gripper.stl" scale="0.01 0.01 0.01"/>
+    </geometry>
+  </collision>
+</link>
+<joint name="joint_1" type="revolute">
   <origin xyz="-0.1101 0.00635 -0.0551" rpy="0 0 0"/>
   <parent link="base_link"/>
@@ -178,9 +209,10 @@
   <limit upper="1.570796" lower="-1.570796" effort="100" velocity="100"/>
 </joint>
-<joint name="joint_3" type="continuous">
+<joint name="joint_3" type="revolute">
   <origin xyz="0.0 0.089 0.003" rpy="0 0 0"/>
   <parent link="link_2"/>
   <child link="link_3"/>
   <axis xyz="-0.0 1.0 -0.0"/>
+  <limit upper="3.14" lower="-3.14" effort="100" velocity="100"/>
 </joint>
 <joint name="joint_4" type="revolute">
@@ -191,9 +223,10 @@
   <limit upper="1.919862" lower="-1.919862" effort="100" velocity="100"/>
 </joint>
-<joint name="joint_5" type="continuous">
+<joint name="joint_5" type="revolute">
   <origin xyz="0.0 0.089 0.003" rpy="0 0 0"/>
   <parent link="link_4"/>
   <child link="link_5"/>
   <axis xyz="-0.0 1.0 -0.0"/>
+  <limit upper="3.14" lower="-3.14" effort="100" velocity="100"/>
 </joint>
 <joint name="joint_6" type="revolute">
@@ -204,9 +237,10 @@
   <limit upper="1.919862" lower="-1.919862" effort="100" velocity="100"/>
 </joint>
-<joint name="joint_7" type="continuous">
+<joint name="joint_7" type="revolute">
   <origin xyz="0.0 0.089 0.003" rpy="0 0 0"/>
   <parent link="link_6"/>
   <child link="gripper"/>
   <axis xyz="-0.0 1.0 -0.0"/>
+  <limit upper="3.14" lower="-3.14" effort="100" velocity="100"/>
 </joint>
 </robot>

Commit message: Gripper works

File: arm2v4_description/urdf/arm2v4.urdf.xacro (robot description, xacro)
@@ -177,4 +177,5 @@
   </collision>
 </link>
+<!--
 <link name="gripper">
   <inertial>
@@ -194,4 +195,105 @@
     <geometry>
       <mesh filename="package://arm2v4_description/meshes/gripper.stl" scale="0.01 0.01 0.01"/>
+    </geometry>
+  </collision>
+</link>
+-->
+<link name="gripper">
+  <inertial>
+    <origin xyz="-7.99617922246049e-05 -9.373301345926424e-05 0.022688831485682622" rpy="0 0 0"/>
+    <mass value="0.06230882557508056"/>
+    <inertia ixx="2e-05" iyy="2e-05" izz="1.8e-05" ixy="0.0" iyz="-0.0" ixz="0.0"/>
+  </inertial>
+  <visual>
+    <origin xyz="0 0 0" rpy="0 0 0"/>
+    <geometry>
+      <mesh filename="package://arm2v4_description/meshes/gripper_base.stl" scale="0.01 0.01 0.01"/>
+    </geometry>
+    <material name="silver"/>
+  </visual>
+  <collision>
+    <origin xyz="0 0 0" rpy="0 0 0"/>
+    <geometry>
+      <mesh filename="package://arm2v4_description/meshes/gripper_base.stl" scale="0.01 0.01 0.01"/>
+    </geometry>
+  </collision>
+</link>
+<link name="finger_1">
+  <inertial>
+    <origin xyz="-0.008642610431029825 -0.0223485533956419 0.01797350009267279" rpy="0 0 0"/>
+    <mass value="0.00589987703289726"/>
+    <inertia ixx="2e-06" iyy="1e-06" izz="1e-06" ixy="-0.0" iyz="1e-06" ixz="0.0"/>
+  </inertial>
+  <visual>
+    <origin xyz="-0.005959 0.022452 -0.054853" rpy="0 0 0"/>
+    <geometry>
+      <mesh filename="package://arm2v4_description/meshes/finger_1.stl" scale="0.01 0.01 0.01"/>
+    </geometry>
+    <material name="silver"/>
+  </visual>
+  <collision>
+    <origin xyz="-0.005959 0.022452 -0.054853" rpy="0 0 0"/>
+    <geometry>
+      <mesh filename="package://arm2v4_description/meshes/finger_1.stl" scale="0.01 0.01 0.01"/>
+    </geometry>
+  </collision>
+</link>
+<link name="finger_2">
+  <inertial>
+    <origin xyz="-0.023075113605405432 0.003290870425902617 0.016944927949491317" rpy="0 0 0"/>
+    <mass value="0.005899814079558049"/>
+    <inertia ixx="1e-06" iyy="2e-06" izz="1e-06" ixy="-0.0" iyz="0.0" ixz="1e-06"/>
+  </inertial>
+  <visual>
+    <origin xyz="0.023955 0.005611 -0.053852" rpy="0 0 0"/>
+    <geometry>
+      <mesh filename="package://arm2v4_description/meshes/finger_2.stl" scale="0.01 0.01 0.01"/>
+    </geometry>
+    <material name="silver"/>
+  </visual>
+  <collision>
+    <origin xyz="0.023955 0.005611 -0.053852" rpy="0 0 0"/>
+    <geometry>
+      <mesh filename="package://arm2v4_description/meshes/finger_2.stl" scale="0.01 0.01 0.01"/>
+    </geometry>
+  </collision>
+</link>
+<link name="finger_3">
+  <inertial>
+    <origin xyz="0.008090867314456025 0.02343237115984798 0.016811323538146863" rpy="0 0 0"/>
+    <mass value="0.005899939849310272"/>
+    <inertia ixx="2e-06" iyy="1e-06" izz="1e-06" ixy="-0.0" iyz="-1e-06" ixz="0.0"/>
+  </inertial>
+  <visual>
+    <origin xyz="0.007093 -0.024302 -0.053188" rpy="0 0 0"/>
+    <geometry>
+      <mesh filename="package://arm2v4_description/meshes/finger_3.stl" scale="0.01 0.01 0.01"/>
+    </geometry>
+    <material name="silver"/>
+  </visual>
+  <collision>
+    <origin xyz="0.007093 -0.024302 -0.053188" rpy="0 0 0"/>
+    <geometry>
+      <mesh filename="package://arm2v4_description/meshes/finger_3.stl" scale="0.01 0.01 0.01"/>
+    </geometry>
+  </collision>
+</link>
+<link name="finger_4">
+  <inertial>
+    <origin xyz="0.022522095224022032 -0.0022060565296590394 0.017840959663214417" rpy="0 0 0"/>
+    <mass value="0.005899858594402945"/>
+    <inertia ixx="1e-06" iyy="2e-06" izz="1e-06" ixy="-0.0" iyz="-0.0" ixz="-1e-06"/>
+  </inertial>
+  <visual>
+    <origin xyz="-0.022822 -0.00746 -0.054188" rpy="0 0 0"/>
+    <geometry>
+      <mesh filename="package://arm2v4_description/meshes/finger_4.stl" scale="0.01 0.01 0.01"/>
+    </geometry>
+    <material name="silver"/>
+  </visual>
+  <collision>
+    <origin xyz="-0.022822 -0.00746 -0.054188" rpy="0 0 0"/>
+    <geometry>
+      <mesh filename="package://arm2v4_description/meshes/finger_4.stl" scale="0.01 0.01 0.01"/>
     </geometry>
   </collision>
@@ -240,9 +342,38 @@
 </joint>
 <joint name="joint_7" type="revolute">
-  <origin xyz="0.0 0.089 0.003" rpy="0 0 0"/>
+ <!-- <origin xyz="0.0 0.089 0.003" rpy="0 0 0"/>-->
+  <origin xyz="0.0 0.09 0.0" rpy="-1.53 0 0"/>
   <parent link="link_6"/>
   <child link="gripper"/>
-  <axis xyz="-0.0 1.0 -0.0"/>
+  <axis xyz="-0.0 0.0 1.0"/>
   <limit upper="3.14" lower="-3.14" effort="100" velocity="100"/>
 </joint>
+<joint name="gripper_joint_1" type="revolute">
+  <origin xyz="0.005959 -0.022452 0.054853" rpy="0 0 0"/>
+  <parent link="gripper"/>
+  <child link="finger_1"/>
+  <axis xyz="0.999727 0.017623 0.01534"/>
+  <limit upper="0.0" lower="-1.134464" effort="100" velocity="100"/>
+</joint>
+<joint name="gripper_joint_2" type="revolute">
+  <origin xyz="-0.023955 -0.005611 0.053852" rpy="0 0 0"/>
+  <parent link="gripper"/>
+  <child link="finger_2"/>
+  <axis xyz="0.017134 -0.999359 0.031436"/>
+  <limit upper="0.0" lower="-1.134464" effort="100" velocity="100"/>
+</joint>
+<joint name="gripper_joint_3" type="revolute">
+  <origin xyz="-0.007093 0.024302 0.053188" rpy="0 0 0"/>
+  <parent link="gripper"/>
+  <child link="finger_3"/>
+  <axis xyz="-0.999727 -0.017623 -0.01534"/>
+  <limit upper="0.0" lower="-1.134464" effort="100" velocity="100"/>
+</joint>
+<joint name="gripper_joint_4" type="revolute">
+  <origin xyz="0.022822 0.00746 0.054188" rpy="0 0 0"/>
+  <parent link="gripper"/>
+  <child link="finger_4"/>
+  <axis xyz="-0.017134 0.999359 -0.031436"/>
+  <limit upper="0.0" lower="-1.134464" effort="100" velocity="100"/>
+</joint>
 </robot>

Commit message: Redid control system

File: arm2v4_description/urdf/arm2v4.urdf.xacro (robot description, xacro)
@@ -30,4 +30,5 @@
   <origin xyz="0 0 0" rpy="1.57 0 0"/>
 </joint>
+  <!--
   <link name="top_plate">
     <inertial>
@@ -36,5 +37,4 @@
         <inertia ixx="0.010238" iyy="0.01139" izz="0.021617" ixy="-0.0" iyz="0.0" ixz="0.0"/>
     </inertial>
-    <!--
     <visual>
         <origin xyz="0 0 0" rpy="0 0 0"/>
@@ -44,5 +44,4 @@
         <material name="silver"/>
     </visual>
-    -->
     <collision>
         <origin xyz="0 0 0.279654" rpy="0 0 0"/>
@@ -52,4 +51,6 @@
     </collision>
   </link>
+  -->
+  <!--
   <joint name="top_connector" type="fixed">
     <parent link="world"/>
@@ -57,4 +58,5 @@
     <origin xyz="0 0 0.279654" rpy="0 0 0"/>
   </joint>
+  -->
 <link name="link_1">
   <inertial>
@@ -299,10 +301,10 @@
   </collision>
 </link>
-<joint name="joint_1" type="revolute">
-  <origin xyz="-0.1101 0.00635 -0.0551" rpy="0 0 0"/>
+<joint name="joint_1" type="continuous">
+  <origin xyz="-0.1101 0.02 -0.0551" rpy="0 0 0"/>
   <parent link="base_link"/>
   <child link="link_1"/>
   <axis xyz="-0.0 -1.0 0.0"/>
-  <limit upper="3.141593" lower="-1.047198" effort="100" velocity="100"/>
+  <!--<limit upper="3.141593" lower="-3.141593" effort="100" velocity="100"/>-->
 </joint>
 <joint name="joint_2" type="revolute">
@@ -313,10 +315,10 @@
   <limit upper="1.570796" lower="-1.570796" effort="100" velocity="100"/>
 </joint>
-<joint name="joint_3" type="revolute">
+<joint name="joint_3" type="continuous">
   <origin xyz="0.0 0.089 0.003" rpy="0 0 0"/>
   <parent link="link_2"/>
   <child link="link_3"/>
   <axis xyz="-0.0 1.0 -0.0"/>
-  <limit upper="3.14" lower="-3.14" effort="100" velocity="100"/>
+  <!--<limit upper="3.14" lower="-3.14" effort="100" velocity="100"/>-->
 </joint>
 <joint name="joint_4" type="revolute">
@@ -327,10 +329,10 @@
   <limit upper="1.919862" lower="-1.919862" effort="100" velocity="100"/>
 </joint>
-<joint name="joint_5" type="revolute">
+<joint name="joint_5" type="continuous">
   <origin xyz="0.0 0.089 0.003" rpy="0 0 0"/>
   <parent link="link_4"/>
   <child link="link_5"/>
   <axis xyz="-0.0 1.0 -0.0"/>
-  <limit upper="3.14" lower="-3.14" effort="100" velocity="100"/>
+  <!--<limit upper="3.14" lower="-3.14" effort="100" velocity="100"/>-->
 </joint>
 <joint name="joint_6" type="revolute">
@@ -341,5 +343,5 @@
   <limit upper="1.919862" lower="-1.919862" effort="100" velocity="100"/>
 </joint>
-<joint name="joint_7" type="revolute">
+<joint name="joint_7" type="continuous">
  <!-- <origin xyz="0.0 0.089 0.003" rpy="0 0 0"/>-->
   <origin xyz="0.0 0.09 0.0" rpy="-1.53 0 0"/>
@@ -347,5 +349,5 @@
   <child link="gripper"/>
   <axis xyz="-0.0 0.0 1.0"/>
-  <limit upper="3.14" lower="-3.14" effort="100" velocity="100"/>
+  <!--<limit upper="3.14" lower="-3.14" effort="100" velocity="100"/>-->
 </joint>
 <joint name="gripper_joint_1" type="revolute">

Commit message: Sped up sim

File: arm2v4_description/urdf/arm2v4.urdf.xacro (robot description, xacro)
@@ -1,4 +1,8 @@
 <?xml version="1.0" ?>
 <robot name="arm2v4" xmlns:xacro="http://www.ros.org/wiki/xacro">
+<xacro:arg name="include_base_plate" default="false"/>
+<xacro:arg name="arm" default="ARM1"/>
+<!-- Convert arg to property -->
+<xacro:property name="arm" value="$(arg arm)"/>
 <material name="silver">
   <color rgba="0.700 0.700 0.700 1.000" />
@@ -6,24 +10,24 @@
 <link name="world"/>
 <link name="base_link">
-  <!--
-  <inertial>
-    <origin xyz="-0.01036605995280163 0.008118725780222396 -0.010698521307181049" rpy="0 0 0"/>
-    <mass value="0.6714813076324946"/>
-    <inertia ixx="0.004693" iyy="0.009008" izz="0.004597" ixy="0.000126" iyz="0.000275" ixz="-0.00051"/>
-  </inertial>
-  <visual>
-    <origin xyz="0 0 0" rpy="0 0 0"/>
-    <geometry>
-      <mesh filename="package://arm2v4_description/meshes/base_link.stl" scale="0.01 0.01 0.01"/>
-    </geometry>
-    <material name="silver"/>
-  </visual>
-  <collision>
-    <origin xyz="0 0 0" rpy="0 0 0"/>
-    <geometry>
-      <mesh filename="package://arm2v4_description/meshes/base_link.stl" scale="0.01 0.01 0.01"/>
-    </geometry>
-  </collision>
-  -->
+  <xacro:if value="$(arg include_base_plate)">
+    <inertial>
+      <origin xyz="-0.01036605995280163 0.008118725780222396 -0.010698521307181049" rpy="0 0 0"/>
+      <mass value="0.6714813076324946"/>
+      <inertia ixx="0.004693" iyy="0.009008" izz="0.004597" ixy="0.000126" iyz="0.000275" ixz="-0.00051"/>
+    </inertial>
+    <visual>
+      <origin xyz="0 0 0" rpy="0 0 0"/>
+      <geometry>
+        <mesh filename="package://arm2v4_description/meshes/base_link.stl" scale="0.01 0.01 0.01"/>
+      </geometry>
+      <material name="silver"/>
+    </visual>
+    <collision>
+      <origin xyz="0 0 0" rpy="0 0 0"/>
+      <geometry>
+        <mesh filename="package://arm2v4_description/meshes/base_link.stl" scale="0.01 0.01 0.01"/>
+      </geometry>
+    </collision>
+  </xacro:if>
 </link>
 <joint name="world_joint" type="fixed">
@@ -304,5 +308,10 @@
 </link>
 <joint name="joint_1" type="continuous">
-  <origin xyz="-0.1101 0.02 -0.0551" rpy="0 0 0"/>
+  <xacro:if value="${arm == 'ARM1'}">
+    <origin xyz="-0.1101 0.007 -0.0551" rpy="0 0 0"/>
+  </xacro:if>
+  <xacro:unless value="${arm == 'ARM1'}">
+    <origin xyz="0.0551 0.007 0.1101" rpy="0 -1.57 0"/>
+  </xacro:unless>
   <parent link="base_link"/>
   <child link="link_1"/>
