Commit message: Arms working

File: arm2v4_description/urdf/arm2v4.urdf.xacro (robot description, xacro)
@@ -221,9 +221,15 @@
   </collision>
 </link>
+<!-- The RPY for these joints must be changed to set start config
+     Notice for each joint the values are repeated this is so the arm
+     can be aware of the other arm
+     CAUTION: Make sure you set R1 and R2 arm2v4_body.xml to match -->
 <joint name="${arm}joint_1" type="continuous">
   <xacro:if value="${namespace == 'ARM1'}">
+    <!-- Set ARM1 -->
     <xacro:if value="${arm == ''}">
       <origin xyz="-0.1101 0.007 -0.0551" rpy="0 1.57 0"/>
     </xacro:if>
+    <!-- Set ARM2 -->
     <xacro:unless value="${arm == ''}">
       <origin xyz="0.0551 0.007 0.1101" rpy="0 0 0"/>
@@ -232,7 +238,9 @@
   <xacro:if value="${namespace == 'ARM2'}">
     <xacro:if value="${arm == ''}">
+    <!-- Set ARM2 -->
       <origin xyz="0.0551 0.007 0.1101" rpy="0 0 0"/>
     </xacro:if>
     <xacro:unless value="${arm == ''}">
+    <!-- Set ARM1 -->
       <origin xyz="-0.1101 0.007 -0.0551" rpy="0 1.57 0"/>
     </xacro:unless>
@@ -251,5 +259,24 @@
 </joint>
 <joint name="${arm}joint_3" type="continuous">
-  <origin xyz="-0.018 0.089 0" rpy="0 0 0"/>
+  <xacro:if value="${namespace == 'ARM1'}">
+    <!-- Set ARM1 -->
+    <xacro:if value="${arm == ''}">
+      <origin xyz="-0.018 0.089 0" rpy="0 0 0"/>
+    </xacro:if>
+    <!-- Set ARM2 -->
+    <xacro:unless value="${arm == ''}">
+      <origin xyz="-0.018 0.089 0" rpy="0 -1.57 0"/>
+    </xacro:unless>
+  </xacro:if>
+  <xacro:if value="${namespace == 'ARM2'}">
+    <!-- Set ARM2 -->
+    <xacro:if value="${arm == ''}">
+      <origin xyz="-0.018 0.089 0" rpy="0 -1.57 0"/>
+    </xacro:if>
+    <!-- Set ARM1 -->
+    <xacro:unless value="${arm == ''}">
+      <origin xyz="-0.018 0.089 0" rpy="0 0 0"/>
+    </xacro:unless>
+  </xacro:if>
   <parent link="${arm}link_2"/>
   <child link="${arm}link_3"/>
@@ -258,9 +285,31 @@
 </joint>
 <joint name="${arm}joint_4" type="revolute">
-  <origin xyz="0.018 0.036618 0" rpy="0 0 0"/>
+  <xacro:if value="${namespace == 'ARM1'}">
+    <!-- Set ARM1 -->
+    <xacro:if value="${arm == ''}">
+      <origin xyz="0.018 0.036618 0" rpy="0 0 0"/>
+      <limit upper="1.919862" lower="-1.919862" effort="100" velocity="100"/>
+    </xacro:if>
+    <!-- Set ARM2 -->
+    <xacro:unless value="${arm == ''}">
+      <origin xyz="0.018 0.036618 0" rpy="1.309 0 0"/>
+      <limit upper="3.316" lower="-0.523" effort="100" velocity="100"/>
+    </xacro:unless>
+  </xacro:if>
+  <xacro:if value="${namespace == 'ARM2'}">
+    <!-- Set ARM2 -->
+    <xacro:if value="${arm == ''}">
+      <origin xyz="0.018 0.036618 0" rpy="1.309 0 0"/>
+      <limit upper="3.316" lower="-0.523" effort="100" velocity="100"/>
+    </xacro:if>
+    <!-- Set ARM1 -->
+    <xacro:unless value="${arm == ''}">
+      <origin xyz="0.018 0.036618 0" rpy="0 0 0"/>
+       <limit upper="1.919862" lower="-1.919862" effort="100" velocity="100"/>
+    </xacro:unless>
+  </xacro:if>
   <parent link="${arm}link_3"/>
   <child link="${arm}link_4"/>
   <axis xyz="-1.0 -0.0 0.0"/>
-  <limit upper="1.919862" lower="-1.919862" effort="100" velocity="100"/>
 </joint>
 <joint name="${arm}joint_5" type="continuous">
@@ -272,9 +321,31 @@
 </joint>
 <joint name="${arm}joint_6" type="revolute">
-  <origin xyz="0.018 0.036617 0" rpy="0 0 0"/>
+  <xacro:if value="${namespace == 'ARM1'}">
+    <!-- Set ARM1 -->
+    <xacro:if value="${arm == ''}">
+      <origin xyz="0.018 0.036617 0" rpy="0 0 0"/>
+      <limit upper="1.919862" lower="-1.919862" effort="100" velocity="100"/>
+    </xacro:if>
+    <!-- Set ARM2 -->
+    <xacro:unless value="${arm == ''}">
+      <origin xyz="0.018 0.036617 0" rpy="1.745 0 0"/>
+      <limit upper="3.316" lower="-0.523" effort="100" velocity="100"/>
+    </xacro:unless>
+  </xacro:if>
+  <xacro:if value="${namespace == 'ARM2'}">
+    <!-- Set ARM2 -->
+    <xacro:if value="${arm == ''}">
+      <origin xyz="0.018 0.036617 0" rpy="1.745 0 0"/>
+      <limit upper="3.316" lower="-0.523" effort="100" velocity="100"/>
+    </xacro:if>
+    <!-- Set ARM1 -->
+    <xacro:unless value="${arm == ''}">
+      <origin xyz="0.018 0.036617 0" rpy="0 0 0"/>
+      <limit upper="1.919862" lower="-1.919862" effort="100" velocity="100"/>
+    </xacro:unless>
+  </xacro:if>
   <parent link="${arm}link_5"/>
   <child link="${arm}link_6"/>
   <axis xyz="-1.0 -0.0 0.0"/>
-  <limit upper="1.919862" lower="-1.919862" effort="100" velocity="100"/>
 </joint>
 <joint name="${arm}joint_7" type="continuous">
@@ -287,5 +358,5 @@
 </joint>
 <joint name="${arm}gripper_joint_1" type="revolute">
-  <origin xyz="0.006125 0.0535 0.0235" rpy="-1.53 0 0"/>
+  <origin xyz="0.006125 0.0535 0.0235" rpy="-2.53 0 0"/>
   <parent link="${arm}gripper"/>
   <child link="${arm}finger_1"/>
@@ -294,5 +365,5 @@
 </joint>
 <joint name="${arm}gripper_joint_2" type="revolute">
-  <origin xyz="-0.0235 0.0535 0.006125" rpy="-1.53 0 0"/>
+  <origin xyz="-0.0235 0.0535 0.006125" rpy="-1.53 0 -1"/>
   <parent link="${arm}gripper"/>
   <child link="${arm}finger_2"/>
@@ -301,5 +372,5 @@
 </joint>
 <joint name="${arm}gripper_joint_3" type="revolute">
-  <origin xyz="-0.006125 0.0535 -0.0235" rpy="-1.53 0 0"/>
+  <origin xyz="-0.006125 0.0535 -0.0235" rpy="-0.53 0 0"/>
   <parent link="${arm}gripper"/>
   <child link="${arm}finger_3"/>
@@ -308,5 +379,5 @@
 </joint>
 <joint name="${arm}gripper_joint_4" type="revolute">
-  <origin xyz="0.0235 0.0535 -0.006125" rpy="-1.53 0 0"/>
+  <origin xyz="0.0235 0.0535 -0.006125" rpy="-1.53 0 1"/>
   <parent link="${arm}gripper"/>
   <child link="${arm}finger_4"/>

File: arm2v4_description/urdf/dual_arm2v4.urdf.xacro (robot description, xacro)
@@ -25,5 +25,5 @@
       <origin xyz="0 0 0" rpy="0 0 0"/>
       <geometry>
-        <mesh filename="package://arm2v4_description/meshes/base_link.stl" scale="0.01 0.01 0.01"/>
+        <mesh filename="package://arm2v4_description/meshes/base_link_full.stl" scale="0.01 0.01 0.01"/>
       </geometry>
       <material name="silver"/>
@@ -32,5 +32,5 @@
       <origin xyz="0 0 0" rpy="0 0 0"/>
       <geometry>
-        <mesh filename="package://arm2v4_description/meshes/base_link.stl" scale="0.01 0.01 0.01"/>
+        <mesh filename="package://arm2v4_description/meshes/base_link_full.stl" scale="0.01 0.01 0.01"/>
       </geometry>
     </collision>

Commit message: update that is probably overdue

File: arm2v4_description/urdf/arm2v4.urdf.xacro (robot description, xacro)
@@ -252,5 +252,25 @@
 </joint>
 <joint name="${arm}joint_2" type="revolute">
-  <origin xyz="0.018 0.035617 0" rpy="0 0 0"/>
+  <!--<origin xyz="0.018 0.035617 0" rpy="0.0698132 0 0"/>-->
+  <xacro:if value="${namespace == 'ARM1'}">
+    <!-- Set ARM1 -->
+    <xacro:if value="${arm == ''}">
+      <origin xyz="0.018 0.035617 0" rpy="0.0698132 0 0"/>
+    </xacro:if>
+  <!-- Set ARM2 -->
+    <xacro:unless value="${arm == ''}">
+      <origin xyz="0.018 0.035617 0" rpy="-0.0698132 0 0"/>
+    </xacro:unless>
+  </xacro:if>
+  <xacro:if value="${namespace == 'ARM2'}">
+    <!-- Set ARM2 -->
+    <xacro:if value="${arm == ''}">
+      <origin xyz="0.018 0.035617 0" rpy="-0.0698132 0 0"/>
+    </xacro:if>
+    <!-- Set ARM1 -->
+    <xacro:unless value="${arm == ''}">
+      <origin xyz="0.018 0.035617 0" rpy="0.0698132 0 0"/>
+    </xacro:unless>
+  </xacro:if>
   <parent link="${arm}link_1"/>
   <child link="${arm}link_2"/>
@@ -262,19 +282,19 @@
     <!-- Set ARM1 -->
     <xacro:if value="${arm == ''}">
-      <origin xyz="-0.018 0.089 0" rpy="0 0 0"/>
-    </xacro:if>
-    <!-- Set ARM2 -->
-    <xacro:unless value="${arm == ''}">
-      <origin xyz="-0.018 0.089 0" rpy="0 -1.57 0"/>
-    </xacro:unless>
-  </xacro:if>
-  <xacro:if value="${namespace == 'ARM2'}">
-    <!-- Set ARM2 -->
-    <xacro:if value="${arm == ''}">
-      <origin xyz="-0.018 0.089 0" rpy="0 -1.57 0"/>
-    </xacro:if>
-    <!-- Set ARM1 -->
-    <xacro:unless value="${arm == ''}">
-      <origin xyz="-0.018 0.089 0" rpy="0 0 0"/>
+      <origin xyz="-0.018 0.089 0" rpy="0 1.663222557 0"/>
+    </xacro:if>
+    <!-- Set ARM2 -->
+    <xacro:unless value="${arm == ''}">
+      <origin xyz="-0.018 0.089 0" rpy="0 -0.24242623 0"/>
+    </xacro:unless>
+  </xacro:if>
+  <xacro:if value="${namespace == 'ARM2'}">
+    <!-- Set ARM2 -->
+    <xacro:if value="${arm == ''}">
+      <origin xyz="-0.018 0.089 0" rpy="0 -0.24242623 0"/>
+    </xacro:if>
+    <!-- Set ARM1 -->
+    <xacro:unless value="${arm == ''}">
+      <origin xyz="-0.018 0.089 0" rpy="0 1.663222557 0"/>
     </xacro:unless>
   </xacro:if>
@@ -288,23 +308,23 @@
     <!-- Set ARM1 -->
     <xacro:if value="${arm == ''}">
-      <origin xyz="0.018 0.036618 0" rpy="0 0 0"/>
-      <limit upper="1.919862" lower="-1.919862" effort="100" velocity="100"/>
-    </xacro:if>
-    <!-- Set ARM2 -->
-    <xacro:unless value="${arm == ''}">
-      <origin xyz="0.018 0.036618 0" rpy="1.309 0 0"/>
-      <limit upper="3.316" lower="-0.523" effort="100" velocity="100"/>
-    </xacro:unless>
-  </xacro:if>
-  <xacro:if value="${namespace == 'ARM2'}">
-    <!-- Set ARM2 -->
-    <xacro:if value="${arm == ''}">
-      <origin xyz="0.018 0.036618 0" rpy="1.309 0 0"/>
-      <limit upper="3.316" lower="-0.523" effort="100" velocity="100"/>
-    </xacro:if>
-    <!-- Set ARM1 -->
-    <xacro:unless value="${arm == ''}">
-      <origin xyz="0.018 0.036618 0" rpy="0 0 0"/>
-       <limit upper="1.919862" lower="-1.919862" effort="100" velocity="100"/>
+      <origin xyz="0.018 0.036618 0" rpy="-1.664346 0 0"/>
+      <limit upper="0.0872665" lower="-3.41" effort="100" velocity="100"/>
+    </xacro:if>
+    <!-- Set ARM2 -->
+    <xacro:unless value="${arm == ''}">
+      <origin xyz="0.018 0.036618 0" rpy="-1.664346 0 0"/>
+      <limit upper="0.0872665" lower="-3.41" effort="100" velocity="100"/>
+    </xacro:unless>
+  </xacro:if>
+  <xacro:if value="${namespace == 'ARM2'}">
+    <!-- Set ARM2 -->
+    <xacro:if value="${arm == ''}">
+      <origin xyz="0.018 0.036618 0" rpy="-1.664346 0 0"/>
+      <limit upper="0.0872665" lower="-3.41" effort="100" velocity="100"/>
+    </xacro:if>
+    <!-- Set ARM1 -->
+    <xacro:unless value="${arm == ''}">
+      <origin xyz="0.018 0.036618 0" rpy="-1.664346 0 0"/>
+       <limit upper="0.0872665" lower="-3.41" effort="100" velocity="100"/>
     </xacro:unless>
   </xacro:if>
@@ -314,5 +334,29 @@
 </joint>
 <joint name="${arm}joint_5" type="continuous">
-  <origin xyz="-0.018 0.089 0" rpy="0 0 0"/>
+  <!--<origin xyz="-0.018 0.089 0" rpy="0 -2.24346 0"/>-->
+  <xacro:if value="${namespace == 'ARM1'}">
+    <!-- Set ARM1 -->
+    <xacro:if value="${arm == ''}">
+      <origin xyz="-0.018 0.089 0" rpy="0 -2.24346 0"/>
+      <limit upper="3.316" lower="-0.523" effort="100" velocity="100"/>
+    </xacro:if>
+    <!-- Set ARM2 -->
+    <xacro:unless value="${arm == ''}">
+      <origin xyz="-0.018 0.089 0" rpy="0 -2.24346 0"/>
+      <limit upper="3.316" lower="-0.523" effort="100" velocity="100"/>
+    </xacro:unless>
+  </xacro:if>
+  <xacro:if value="${namespace == 'ARM2'}">
+    <!-- Set ARM2 -->
+    <xacro:if value="${arm == ''}">
+      <origin xyz="-0.018 0.089 0" rpy="0 -2.24346 0"/>
+      <limit upper="3.316" lower="-0.523" effort="100" velocity="100"/>
+    </xacro:if>
+    <!-- Set ARM1 -->
+    <xacro:unless value="${arm == ''}">
+      <origin xyz="-0.018 0.089 0" rpy="0 -2.24346 0"/>
+      <limit upper="3.316" lower="-0.523" effort="100" velocity="100"/>
+    </xacro:unless>
+  </xacro:if>
   <parent link="${arm}link_4"/>
   <child link="${arm}link_5"/>
@@ -324,23 +368,23 @@
     <!-- Set ARM1 -->
     <xacro:if value="${arm == ''}">
-      <origin xyz="0.018 0.036617 0" rpy="0 0 0"/>
-      <limit upper="1.919862" lower="-1.919862" effort="100" velocity="100"/>
-    </xacro:if>
-    <!-- Set ARM2 -->
-    <xacro:unless value="${arm == ''}">
-      <origin xyz="0.018 0.036617 0" rpy="1.745 0 0"/>
-      <limit upper="3.316" lower="-0.523" effort="100" velocity="100"/>
-    </xacro:unless>
-  </xacro:if>
-  <xacro:if value="${namespace == 'ARM2'}">
-    <!-- Set ARM2 -->
-    <xacro:if value="${arm == ''}">
-      <origin xyz="0.018 0.036617 0" rpy="1.745 0 0"/>
-      <limit upper="3.316" lower="-0.523" effort="100" velocity="100"/>
-    </xacro:if>
-    <!-- Set ARM1 -->
-    <xacro:unless value="${arm == ''}">
-      <origin xyz="0.018 0.036617 0" rpy="0 0 0"/>
-      <limit upper="1.919862" lower="-1.919862" effort="100" velocity="100"/>
+      <origin xyz="0.018 0.036617 0" rpy="1.6281267 0 0"/>
+      <limit upper="3.14" lower="0" effort="100" velocity="100"/>
+    </xacro:if>
+    <!-- Set ARM2 -->
+    <xacro:unless value="${arm == ''}">
+      <origin xyz="0.018 0.036617 0" rpy="1.6281267 0 0"/>
+      <limit upper="3.14" lower="0" effort="100" velocity="100"/>
+    </xacro:unless>
+  </xacro:if>
+  <xacro:if value="${namespace == 'ARM2'}">
+    <!-- Set ARM2 -->
+    <xacro:if value="${arm == ''}">
+      <origin xyz="0.018 0.036617 0" rpy="1.6281267 0 0"/>
+      <limit upper="3.14" lower="0" effort="100" velocity="100"/>
+    </xacro:if>
+    <!-- Set ARM1 -->
+    <xacro:unless value="${arm == ''}">
+      <origin xyz="0.018 0.036617 0" rpy="1.6281267 0 0"/>
+      <limit upper="3.14" lower="0" effort="100" velocity="100"/>
     </xacro:unless>
   </xacro:if>

File: arm2v4_description/urdf/dual_arm2v4.urdf.xacro (robot description, xacro)
@@ -50,5 +50,5 @@
     </inertial>
     <visual>
-        <origin xyz="0 0 0" rpy="0 0 3.14"/>
+        <origin xyz="0 0 0.0127" rpy="0 0 3.14"/>
         <geometry>
         <mesh filename="package://arm2d2_v2_description/meshes/base_plate.stl" scale="0.001 0.001 0.001"/>
@@ -57,5 +57,5 @@
     </visual>
     <collision>
-        <origin xyz="0 0.01 0" rpy="0 0 3.14"/>
+        <origin xyz="0 0.01 0.0127" rpy="0 0 3.14"/>
         <geometry>
         <mesh filename="package://arm2d2_v2_description/meshes/base_plate.stl" scale="0.001 0.001 0.001"/>

Commit message: state machine updates ready-ish for merge

File: arm2v4_description/urdf/arm2v4.urdf.xacro (robot description, xacro)
@@ -225,13 +225,15 @@
      can be aware of the other arm
      CAUTION: Make sure you set R1 and R2 arm2v4_body.xml to match -->
-<joint name="${arm}joint_1" type="continuous">
+<joint name="${arm}joint_1" type="revolute">
   <xacro:if value="${namespace == 'ARM1'}">
     <!-- Set ARM1 -->
     <xacro:if value="${arm == ''}">
       <origin xyz="-0.1101 0.007 -0.0551" rpy="0 1.57 0"/>
+      <limit upper="0.436332" lower="-1.22173" effort="100" velocity="100"/>
     </xacro:if>
     <!-- Set ARM2 -->
     <xacro:unless value="${arm == ''}">
       <origin xyz="0.0551 0.007 0.1101" rpy="0 0 0"/>
+      <limit upper="1.22173" lower="-0.436332" effort="100" velocity="100"/>
     </xacro:unless>
   </xacro:if>
@@ -240,8 +242,10 @@
     <!-- Set ARM2 -->
       <origin xyz="0.0551 0.007 0.1101" rpy="0 0 0"/>
+      <limit upper="1.22173" lower="-0.436332" effort="100" velocity="100"/>
     </xacro:if>
     <xacro:unless value="${arm == ''}">
     <!-- Set ARM1 -->
       <origin xyz="-0.1101 0.007 -0.0551" rpy="0 1.57 0"/>
+      <limit upper="0.436332" lower="-1.22173" effort="100" velocity="100"/>
     </xacro:unless>
   </xacro:if>
@@ -249,5 +253,4 @@
   <child link="${arm}link_1"/>
   <axis xyz="-0.0 -1.0 0.0"/>
-  <!--<limit upper="3.141593" lower="-3.141593" effort="100" velocity="100"/>-->
 </joint>
 <joint name="${arm}joint_2" type="revolute">

Commit message: SM is ready for hardware integration

File: arm2v4_description/urdf/arm2v4.urdf.xacro (robot description, xacro)
@@ -259,19 +259,19 @@
     <!-- Set ARM1 -->
     <xacro:if value="${arm == ''}">
-      <origin xyz="0.018 0.035617 0" rpy="0.0698132 0 0"/>
+      <origin xyz="0.018 0.035617 0" rpy="0 0 0"/> <!--rpy="0.0698132 0 0"/-->
     </xacro:if>
   <!-- Set ARM2 -->
     <xacro:unless value="${arm == ''}">
-      <origin xyz="0.018 0.035617 0" rpy="-0.0698132 0 0"/>
-    </xacro:unless>
-  </xacro:if>
-  <xacro:if value="${namespace == 'ARM2'}">
-    <!-- Set ARM2 -->
-    <xacro:if value="${arm == ''}">
-      <origin xyz="0.018 0.035617 0" rpy="-0.0698132 0 0"/>
-    </xacro:if>
-    <!-- Set ARM1 -->
-    <xacro:unless value="${arm == ''}">
-      <origin xyz="0.018 0.035617 0" rpy="0.0698132 0 0"/>
+      <origin xyz="0.018 0.035617 0" rpy="0 0 0"/> <!--rpy="-0.0698132 0 0"/-->
+    </xacro:unless>
+  </xacro:if>
+  <xacro:if value="${namespace == 'ARM2'}">
+    <!-- Set ARM2 -->
+    <xacro:if value="${arm == ''}">
+      <origin xyz="0.018 0.035617 0" rpy="0 0 0"/> <!--rpy="-0.0698132 0 0"/-->
+    </xacro:if>
+    <!-- Set ARM1 -->
+    <xacro:unless value="${arm == ''}">
+      <origin xyz="0.018 0.035617 0" rpy="0 0 0"/> <!--rpy="0.0698132 0 0"/-->
     </xacro:unless>
   </xacro:if>
@@ -285,19 +285,19 @@
     <!-- Set ARM1 -->
     <xacro:if value="${arm == ''}">
-      <origin xyz="-0.018 0.089 0" rpy="0 1.663222557 0"/>
-    </xacro:if>
-    <!-- Set ARM2 -->
-    <xacro:unless value="${arm == ''}">
-      <origin xyz="-0.018 0.089 0" rpy="0 -0.24242623 0"/>
-    </xacro:unless>
-  </xacro:if>
-  <xacro:if value="${namespace == 'ARM2'}">
-    <!-- Set ARM2 -->
-    <xacro:if value="${arm == ''}">
-      <origin xyz="-0.018 0.089 0" rpy="0 -0.24242623 0"/>
-    </xacro:if>
-    <!-- Set ARM1 -->
-    <xacro:unless value="${arm == ''}">
-      <origin xyz="-0.018 0.089 0" rpy="0 1.663222557 0"/>
+      <origin xyz="-0.018 0.089 0" rpy="0 0 0"/> <!--rpy="0 1.663222557 0"/-->
+    </xacro:if>
+    <!-- Set ARM2 -->
+    <xacro:unless value="${arm == ''}">
+      <origin xyz="-0.018 0.089 0" rpy="0 0 0"/> <!--rpy="0 -0.24242623 0"/-->
+    </xacro:unless>
+  </xacro:if>
+  <xacro:if value="${namespace == 'ARM2'}">
+    <!-- Set ARM2 -->
+    <xacro:if value="${arm == ''}">
+      <origin xyz="-0.018 0.089 0" rpy="0 0 0"/> <!--rpy="0 -0.24242623 0"/-->
+    </xacro:if>
+    <!-- Set ARM1 -->
+    <xacro:unless value="${arm == ''}">
+      <origin xyz="-0.018 0.089 0" rpy="0 0 0"/> <!--rpy="0 1.663222557 0"/-->
     </xacro:unless>
   </xacro:if>
@@ -311,10 +311,10 @@
     <!-- Set ARM1 -->
     <xacro:if value="${arm == ''}">
-      <origin xyz="0.018 0.036618 0" rpy="-1.664346 0 0"/>
+      <origin xyz="0.018 0.036618 0" rpy="0 0 0"/> <!--rpy="-1.664346 0 0"/-->
       <limit upper="0.0872665" lower="-3.41" effort="100" velocity="100"/>
     </xacro:if>
     <!-- Set ARM2 -->
     <xacro:unless value="${arm == ''}">
-      <origin xyz="0.018 0.036618 0" rpy="-1.664346 0 0"/>
+      <origin xyz="0.018 0.036618 0" rpy="0 0 0"/> <!--rpy="-1.664346 0 0"/-->
       <limit upper="0.0872665" lower="-3.41" effort="100" velocity="100"/>
     </xacro:unless>
@@ -323,10 +323,10 @@
     <!-- Set ARM2 -->
     <xacro:if value="${arm == ''}">
-      <origin xyz="0.018 0.036618 0" rpy="-1.664346 0 0"/>
+      <origin xyz="0.018 0.036618 0" rpy="0 0 0"/> <!--rpy="-1.664346 0 0"/-->
       <limit upper="0.0872665" lower="-3.41" effort="100" velocity="100"/>
     </xacro:if>
     <!-- Set ARM1 -->
     <xacro:unless value="${arm == ''}">
-      <origin xyz="0.018 0.036618 0" rpy="-1.664346 0 0"/>
+      <origin xyz="0.018 0.036618 0" rpy="0 0 0"/> <!--rpy="-1.664346 0 0"/-->
        <limit upper="0.0872665" lower="-3.41" effort="100" velocity="100"/>
     </xacro:unless>
@@ -341,10 +341,10 @@
     <!-- Set ARM1 -->
     <xacro:if value="${arm == ''}">
-      <origin xyz="-0.018 0.089 0" rpy="0 -2.24346 0"/>
+      <origin xyz="-0.018 0.089 0" rpy="0 0 0"/> <!--rpy="0 -2.24346 0"/-->
       <limit upper="3.316" lower="-0.523" effort="100" velocity="100"/>
     </xacro:if>
     <!-- Set ARM2 -->
     <xacro:unless value="${arm == ''}">
-      <origin xyz="-0.018 0.089 0" rpy="0 -2.24346 0"/>
+      <origin xyz="-0.018 0.089 0" rpy="0 0 0"/> <!--rpy="0 -2.24346 0"/-->
       <limit upper="3.316" lower="-0.523" effort="100" velocity="100"/>
     </xacro:unless>
@@ -353,10 +353,10 @@
     <!-- Set ARM2 -->
     <xacro:if value="${arm == ''}">
-      <origin xyz="-0.018 0.089 0" rpy="0 -2.24346 0"/>
+      <origin xyz="-0.018 0.089 0" rpy="0 0 0"/> <!--rpy="0 -2.24346 0"/-->
       <limit upper="3.316" lower="-0.523" effort="100" velocity="100"/>
     </xacro:if>
     <!-- Set ARM1 -->
     <xacro:unless value="${arm == ''}">
-      <origin xyz="-0.018 0.089 0" rpy="0 -2.24346 0"/>
+      <origin xyz="-0.018 0.089 0" rpy="0 0 0"/> <!--rpy="0 -2.24346 0"/-->
       <limit upper="3.316" lower="-0.523" effort="100" velocity="100"/>
     </xacro:unless>
@@ -371,23 +371,23 @@
     <!-- Set ARM1 -->
     <xacro:if value="${arm == ''}">
-      <origin xyz="0.018 0.036617 0" rpy="1.6281267 0 0"/>
+      <origin xyz="0.018 0.036617 0" rpy="0 0 0"/> <!--rpy="1.6281267 0 0"/-->
+      <limit upper="1.57" lower="-1.57" effort="100" velocity="100"/>
+    </xacro:if>
+    <!-- Set ARM2 -->
+    <xacro:unless value="${arm == ''}">
+      <origin xyz="0.018 0.036617 0" rpy="0 0 0"/> <!--rpy="1.6281267 0 0"/-->
       <limit upper="3.14" lower="0" effort="100" velocity="100"/>
-    </xacro:if>
-    <!-- Set ARM2 -->
-    <xacro:unless value="${arm == ''}">
-      <origin xyz="0.018 0.036617 0" rpy="1.6281267 0 0"/>
+    </xacro:unless>
+  </xacro:if>
+  <xacro:if value="${namespace == 'ARM2'}">
+    <!-- Set ARM2 -->
+    <xacro:if value="${arm == ''}">
+      <origin xyz="0.018 0.036617 0" rpy="0 0 0"/> <!--rpy="1.6281267 0 0"/-->
       <limit upper="3.14" lower="0" effort="100" velocity="100"/>
-    </xacro:unless>
-  </xacro:if>
-  <xacro:if value="${namespace == 'ARM2'}">
-    <!-- Set ARM2 -->
-    <xacro:if value="${arm == ''}">
-      <origin xyz="0.018 0.036617 0" rpy="1.6281267 0 0"/>
-      <limit upper="3.14" lower="0" effort="100" velocity="100"/>
-    </xacro:if>
-    <!-- Set ARM1 -->
-    <xacro:unless value="${arm == ''}">
-      <origin xyz="0.018 0.036617 0" rpy="1.6281267 0 0"/>
-      <limit upper="3.14" lower="0" effort="100" velocity="100"/>
+    </xacro:if>
+    <!-- Set ARM1 -->
+    <xacro:unless value="${arm == ''}">
+      <origin xyz="0.018 0.036617 0" rpy="0 0 0"/> <!--rpy="1.6281267 0 0"/-->
+      <limit upper="1.57" lower="-1.57" effort="100" velocity="100"/>
     </xacro:unless>
   </xacro:if>

File: arm2v4_description/urdf/dual_arm2v4.urdf.xacro (robot description, xacro)
@@ -15,4 +15,5 @@
 </material>
 <link name="world"/>
+<!---->
 <link name="base_link">
   <xacro:if value="$(arg include_base_plate)">
@@ -22,4 +23,5 @@
       <inertia ixx="0.004693" iyy="0.009008" izz="0.004597" ixy="0.000126" iyz="0.000275" ixz="-0.00051"/>
     </inertial>
+    <!--
     <visual>
       <origin xyz="0 0 0" rpy="0 0 0"/>
@@ -35,4 +37,5 @@
       </geometry>
     </collision>
+    -->
   </xacro:if>
 </link>
